Commit message: Complete fordware position controller in simulation

File: src/description/urdf/servo.urdf.xacro (robot description, xacro)
@@ -1,4 +1,5 @@
 <?xml version="1.0"?>
-<robot name="micro_servo" xmlns:xacro="http://ros.org/wiki/xacro">
+<robot xmlns:xacro="http://ros.org/wiki/xacro">
+  <xacro:macro name="micro_servo" params="parent prefix *origin">
   <!-- Physical Material Macros -->
   <material name="Red">
@@ -22,4 +23,10 @@
   <xacro:property name="rot_link_width" value="0.005" />
   <xacro:property name="rot_link_heigth" value="0.004" />
+  <joint name="${prefix}base_joint" type="fixed">
+    <xacro:insert_block name="origin" />
+    <parent link="${parent}"/>
+    <child link="${prefix}base_link" />
+  </joint>
+  <!-- Base Link -->
   <link name="base_link">
     <visual>
@@ -81,3 +88,4 @@
     <origin xyz="0 0 ${rot_link_heigth}" rpy="0 0 0" />
   </joint>
+</xacro:macro>
 </robot>

Commit message: Set servo joint as revolute

File: src/description/urdf/servo.urdf.xacro (robot description, xacro)
@@ -82,9 +82,10 @@
     </collision>
   </link>
-  <joint name="support_to_rot_link" type="continuous">
+  <joint name="support_to_rot_link" type="revolute">
     <parent link="support_link" />
     <child link="rot_link" />
     <axis xyz="0 0 1"/>
     <origin xyz="0 0 ${rot_link_heigth}" rpy="0 0 0" />
+    <limit lower="0" upper="0" effort="1000" velocity="100"/>
   </joint>
 </xacro:macro>

Commit message: Fixed upper limit revolute joint

File: src/description/urdf/servo.urdf.xacro (robot description, xacro)
@@ -87,5 +87,5 @@
     <axis xyz="0 0 1"/>
     <origin xyz="0 0 ${rot_link_heigth}" rpy="0 0 0" />
-    <limit lower="0" upper="0" effort="1000" velocity="100"/>
+    <limit lower="0" upper="${pi}" effort="1000" velocity="100"/>
   </joint>
 </xacro:macro>
